Commit message: feat: add quadcopter arms using Xacro macros

File: drone_ws/src/drone_description/urdf/drone.urdf.xacro (robot description, xacro)
@@ -1,20 +1,64 @@
 <?xml version="1.0"?>
-<robot xmlns:xacro="http://www.ros.org/wiki/xacro" name="ras_drone"> /el nombre del robot me imagino
-  /estos son los xacros para definir completamente las dimensiones del robot sin necesidad de cambiar todo
+<robot xmlns:xacro="http://www.ros.org/wiki/xacro"
+       name="ras_drone">
   <xacro:property name="body_length" value="0.30"/>
-  <xacro:property name="body_width"  value="0.20"/>
+  <xacro:property name="body_width" value="0.20"/>
   <xacro:property name="body_height" value="0.08"/>
-  <link name="base_link"> /es el componente de la base del robot, mi primer punto de coordenadas
-    <visual> /el como y donde se va a ver
-      <origin xyz="0 0 0" rpy="0 0 0"/> /don de aparece el robot y no se que es rpy
-      <geometry> /la geometria del robot su ancho largo y alto
+  <xacro:property name="arm_length" value="0.22"/>
+  <xacro:property name="arm_width" value="0.025"/>
+  <xacro:property name="arm_height" value="0.025"/>
+  <xacro:property name="arm_radius" value="0.24"/>
+  <link name="base_link">
+    <visual>
+      <geometry>
         <box size="${body_length}
                    ${body_width}
                    ${body_height}"/>
       </geometry>
-      <material name="dark_gray"> /el de que esta hecho con su color y transparencia le puso un nombre y todo
+      <material name="dark_gray">
         <color rgba="0.25 0.28 0.32 1.0"/>
       </material>
     </visual>
   </link>
+  <xacro:macro name="create_arm"
+               params="name x y yaw">
+    <link name="${name}_arm">
+      <visual>
+        <geometry>
+          <box size="${arm_length}
+                     ${arm_width}
+                     ${arm_height}"/>
+        </geometry>
+        <material name="arm_gray">
+          <color rgba="0.65 0.68 0.72 1.0"/>
+        </material>
+      </visual>
+    </link>
+    <joint name="${name}_joint" type="fixed">
+      <parent link="base_link"/>
+      <child link="${name}_arm"/>
+      <origin xyz="${x} ${y} 0"
+              rpy="0 0 ${yaw}"/>
+    </joint>
+  </xacro:macro>
+  <xacro:create_arm
+      name="front_left"
+      x="${arm_radius*cos(pi/4)}"
+      y="${arm_radius*sin(pi/4)}"
+      yaw="${pi/4}"/>
+  <xacro:create_arm
+      name="front_right"
+      x="${arm_radius*cos(-pi/4)}"
+      y="${arm_radius*sin(-pi/4)}"
+      yaw="${-pi/4}"/>
+  <xacro:create_arm
+      name="rear_left"
+      x="${arm_radius*cos(3*pi/4)}"
+      y="${arm_radius*sin(3*pi/4)}"
+      yaw="${3*pi/4}"/>
+  <xacro:create_arm
+      name="rear_right"
+      x="${arm_radius*cos(-3*pi/4)}"
+      y="${arm_radius*sin(-3*pi/4)}"
+      yaw="${-3*pi/4}"/>
 </robot>

Commit message: feat: add quadcopter motors and rotating propellers

File: drone_ws/src/drone_description/urdf/drone.urdf.xacro (robot description, xacro)
@@ -9,4 +9,9 @@
   <xacro:property name="arm_height" value="0.025"/>
   <xacro:property name="arm_radius" value="0.24"/>
+  <xacro:property name="motor_radius" value="0.035"/>
+  <xacro:property name="motor_height" value="0.045"/>
+  <xacro:property name="propeller_length" value="0.18"/>
+  <xacro:property name="propeller_width" value="0.016"/>
+  <xacro:property name="propeller_height" value="0.005"/>
   <link name="base_link">
     <visual>
@@ -42,9 +47,60 @@
     </joint>
   </xacro:macro>
+  <xacro:macro name="create_motor"
+             params="name">
+    <link name="${name}_motor">
+      <visual>
+        <geometry>
+          <cylinder
+            radius="${motor_radius}"
+            length="${motor_height}"/>
+        </geometry>
+        <material name="motor_black">
+          <color rgba="0.12 0.14 0.17 1.0"/>
+        </material>
+      </visual>
+    </link>
+    <joint name="${name}_motor_joint" type="fixed">
+      <parent link="${name}_arm"/>
+      <child link="${name}_motor"/>
+      <origin
+        xyz="${arm_length/2} 0 0.025"
+        rpy="0 0 0"/>
+    </joint>
+      <link name="${name}_propeller">
+      <visual>
+        <geometry>
+          <box size="${propeller_length}
+                     ${propeller_width}
+                     ${propeller_height}"/>
+        </geometry>
+        <material name="propeller_blue">
+          <color rgba="0.15 0.45 0.85 1.0"/>
+        </material>
+      </visual>
+      <visual>
+        <geometry>
+          <box size="${propeller_width}
+                     ${propeller_length}
+                     ${propeller_height}"/>
+        </geometry>
+        <material name="propeller_blue">
+          <color rgba="0.15 0.45 0.85 1.0"/>
+        </material>
+      </visual>
+    </link>
+    <joint name="${name}_propeller_joint"
+           type="continuous">
+      <parent link="${name}_motor"/>
+      <child link="${name}_propeller"/>
+      <origin xyz="0 0 0.035" rpy="0 0 0"/>
+      <axis xyz="0 0 1"/>
+    </joint>
+  </xacro:macro>
   <xacro:create_arm
-      name="front_left"
-      x="${arm_radius*cos(pi/4)}"
-      y="${arm_radius*sin(pi/4)}"
-      yaw="${pi/4}"/>
+        name="front_left"
+        x="${arm_radius*cos(pi/4)}"
+        y="${arm_radius*sin(pi/4)}"
+        yaw="${pi/4}"/>
   <xacro:create_arm
       name="front_right"
@@ -62,3 +118,7 @@
       y="${arm_radius*sin(-3*pi/4)}"
       yaw="${-3*pi/4}"/>
+  <xacro:create_motor name="front_left"/>
+  <xacro:create_motor name="front_right"/>
+  <xacro:create_motor name="rear_left"/>
+  <xacro:create_motor name="rear_right"/>
 </robot>
